File: hardware/hardware/hardware.kicad_pcb (KiCad board)
At the start: 2 copper layers, 34 x 100 mm, 53 parts, among them J1 POWER, J2 SENSOR, J3 RELAY, J4 UART, J5 AVR-ISP-6, K1 FINDER-43.41, Q1 Q_NPN_CBE, Q2 Q_PNP_CBE, Q3 Q_PNP_CBE, Q4 Q_PNP_CBE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

Commit message: pcb
Parts:
- added R22: 100R, Resistor_SMD:R_0805_2012Metric, F.Cu at (161.0, 121.8)
- added REF**: OSHW-Symbol_6.7x6mm_SilkScreen, Symbol:OSHW-Symbol_6.7x6mm_SilkScreen, F.Cu at (144.8, 120.0)
- added REF**: OSHW-Logo2_14.6x12mm_SilkScreen, Symbol:OSHW-Logo2_14.6x12mm_SilkScreen, B.Cu at (175.5, 100.8)
- D3: value LED_STATE -> STAT
- D5, Q2, Q3, Q4, Q6, Q7, R10, R11, R12, R13, R14, R15, R16, R17, R18, R19, R2, R20, R4, R9: moved to B.Cu
- D6: value LED_RELAY -> OUT
- SW1, SW2, SW3: footprint Button_Switch_THT:SW_PUSH_6mm_H5mm -> Button_Switch_SMD:SW_Push_1P1T_NO_6x6mm_H9.5mm
- U1: footprint Package_SO:SO-16_5.3x10.2mm_P1.27mm -> Package_SO:SOIC-16W_5.3x10.2mm_P1.27mm; moved to B.Cu
- moved J3 112.1 mm to (130.2, 86.0), turned to 180 degrees
- moved Y1 100.3 mm to (169.3, 89.8), turned to 0 degrees
- moved U4 93.3 mm to (172.1, 101.2), turned to 180 degrees
- moved J1 89.0 mm to (125.2, 120.3)
- moved J2 88.7 mm to (132.2, 120.3)
- moved J5 85.0 mm to (174.8, 111.5), turned to -90 degrees
- moved K1 76.3 mm to (161.8, 92.5), turned to 180 degrees
- moved D2 75.3 mm to (143.1, 107.8)
- moved SW1 64.0 mm to (128.3, 95.5), turned to 180 degrees
- moved SW2 58.1 mm to (128.3, 104.0), turned to 180 degrees
- moved C3 57.5 mm to (131.6, 99.5), turned to 0 degrees
- moved C4 57.3 mm to (123.7, 109.4), turned to 135 degrees
- moved D1 55.6 mm to (156.2, 121.8), turned to 180 degrees
- moved C6 55.2 mm to (126.8, 104.7)
- moved SW3 55.0 mm to (128.3, 112.5), turned to 0 degrees
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Connections:
- D1 pad 1: +5V -> Net-(D1-K)
- LS1 pad P: +5V -> Net-(D1-K)
Routing:
- net +5V: track 0.00 -> 256.8 mm, vias 0 -> 9
- net Net-(U1-QA): track 0.00 -> 86.4 mm, vias 0 -> 4
- net +12V: track 0.00 -> 77.2 mm, vias 0 -> 3
- net /SW_PLUS: track 0.00 -> 68.1 mm, vias 0 -> 2
- net /SW_SET: track 0.00 -> 66.5 mm, vias 0 -> 2
- net /SW_MINUS: track 0.00 -> 56.0 mm
- net /RELAY: track 0.00 -> 52.9 mm, vias 0 -> 1
- net /DQ: track 0.00 -> 52.3 mm, vias 0 -> 4
- net /DIGIT4: track 0.00 -> 49.2 mm, vias 0 -> 5
- net /DIGIT2: track 0.00 -> 48.0 mm, vias 0 -> 3
- net Net-(D5-A): track 0.00 -> 47.0 mm, vias 0 -> 1
- net Net-(U1-QE): track 0.00 -> 43.3 mm, vias 0 -> 2
- net /BUZZER: track 0.00 -> 42.6 mm, vias 0 -> 5
- net Net-(U4-PD6): track 0.00 -> 42.5 mm
- net /DIGIT3: track 0.00 -> 32.9 mm, vias 0 -> 3
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- added copper zone on B.Cu, net GND
- added copper zone on F.Cu, net GND
Other:
- board size 34 x 100 mm -> 66.5 x 46 mm
- board text added: "+12V"
- board text added: "+5V"
- board text added: "COM"
- board text added: "DQ"
- board text added: "Designed by: Sergey Yarkov"
- board text added: "GND"
- board text added: "ISP"
- board text added: "NC"
- board text added: "NO"
- board text added: "TX"
- board text added: "https://github.com/sergeyyarkov/attiny2313a_thermostat"
